Commit message: Current-Progress

File: Beaker_500ml.urdf (robot description, URDF)
Before this commit: robot beaker_mesh, 1 links, 0 joints
Links:
- link baseLink: geometry collision mesh filename=Beaker_Files/Beaker_500ml.obj scale=0.5 0.5 0.5; visual mesh filename=Beaker_Files/Beaker_500ml.obj scale=0.5 0.5 0.5

Commit message: About to make changes to the rewards function

File: Beaker_500ml.urdf (robot description, URDF)
Before this commit: robot beaker_mesh, 1 links, 0 joints
Links:
- link baseLink: geometry collision mesh filename=Beaker_Files/Beaker.obj scale=0.065 0.065 0.075; visual mesh filename=Beaker_Files/Beaker.obj scale=0.065 0.065 0.075
